Commit message: Add dynamic wheelchair push training task

File: assets/objects/wheelchair/free3d_active_wheelchair/urdf/active_manual_wheelchair.urdf (robot description, URDF)
Before this commit: robot active_manual_wheelchair, 9 links, 8 joints
Links:
- link left_handle_frame: geometry collision box size=0.18 0.055 0.055; visual box size=0.18 0.055 0.055
- link right_handle_frame: geometry collision box size=0.18 0.055 0.055; visual box size=0.18 0.055 0.055

Commit message: Hide wheelchair helper visuals

File: assets/objects/wheelchair/free3d_active_wheelchair/urdf/active_manual_wheelchair.urdf (robot description, URDF)
Before this commit: robot active_manual_wheelchair, 9 links, 8 joints
Links:
- link left_front_caster: geometry collision cylinder length=0.035 radius=0.075
- link left_handle_frame: geometry collision box size=0.18 0.055 0.055
- link left_rear_wheel: geometry collision cylinder length=0.045 radius=0.31
- link right_front_caster: geometry collision cylinder length=0.035 radius=0.075
- link right_handle_frame: geometry collision box size=0.18 0.055 0.055
- link right_rear_wheel: geometry collision cylinder length=0.045 radius=0.31

Commit message: Add wheelchair four-wheel ground bias

File: assets/objects/wheelchair/free3d_active_wheelchair/urdf/active_manual_wheelchair.urdf (robot description, URDF)
Before this commit: robot active_manual_wheelchair, 9 links, 8 joints
Joints:
- joint left_front_caster_joint: origin xyz=0.00 0.00 -0.05 rpy=0 0 0 -> xyz=0.00 0.00 -0.085 rpy=0 0 0
- joint right_front_caster_joint: origin xyz=0.00 0.00 -0.05 rpy=0 0 0 -> xyz=0.00 0.00 -0.085 rpy=0 0 0

Commit message: Align wheelchair handles before hard attachment

File: assets/objects/wheelchair/free3d_active_wheelchair/urdf/active_manual_wheelchair.urdf (robot description, URDF)
Before this commit: robot active_manual_wheelchair, 9 links, 8 joints
Joints:
- joint left_handle_frame_joint: origin xyz=-0.40 0.24 0.88 rpy=0 0 0 -> xyz=-0.40 0.24 0.92029 rpy=0 0 0
- joint right_handle_frame_joint: origin xyz=-0.40 -0.24 0.88 rpy=0 0 0 -> xyz=-0.40 -0.24 0.92029 rpy=0 0 0

Commit message: Clear wheelchair handle collision lanes

File: assets/objects/wheelchair/free3d_active_wheelchair/urdf/active_manual_wheelchair.urdf (robot description, URDF)
Before this commit: robot active_manual_wheelchair, 9 links, 8 joints
Links:
- link base_link: geometry collision box size=0.07 0.32 0.44; collision box size=0.08 0.58 0.08
- link left_handle_frame: geometry collision box size=0.12 0.04 0.04
- link right_handle_frame: geometry collision box size=0.12 0.04 0.04

File: assets/objects/wheelchair/free3d_active_wheelchair/urdf/active_manual_wheelchair_proxy_visual.urdf (robot description, URDF)
Before this commit: robot active_manual_wheelchair_proxy_visual, 9 links, 8 joints
Links:
- link base_link: geometry collision box size=0.07 0.32 0.44; collision box size=0.08 0.58 0.08
- link left_handle_frame: geometry collision box size=0.12 0.04 0.04; visual box size=0.12 0.04 0.04
- link right_handle_frame: geometry collision box size=0.12 0.04 0.04; visual box size=0.12 0.04 0.04
