Commit message: Stabilize wheelchair PhysX rail training

File: assets/objects/wheelchair/free3d_active_wheelchair/urdf/active_manual_wheelchair_x_rail.urdf (robot description, URDF)
Before this commit: robot active_manual_wheelchair_x_rail, 10 links, 9 joints
Joints:
- joint rail_x_joint: limit lower=-1000.0 upper=1000.0 effort=100000.0 velocity=100.0 -> lower=-1000.0 upper=1000.0 effort=500.0 velocity=4.0
